File: pcb/plant-sense.sch (EAGLE design)
At the start: 81 parts, among them CON1 3P-SH-SIDE, CON2 3P-SH-SIDE, CON3 3P-SH-SIDE, CON4 3P-SH-SIDE, Q1 AO3401, T1 BC817, U1 MCP1253-33X50, U15 TP4056, U2 MIC23155, U3 FS312F-G, U4 FS8205, U5 EFM32PG1B200F256GM32, U6 SST26VF016B, U7 RFM69HW, U8 SI7021, X1 40MHz

Commit message: Schematic work
Parts:
- CON1, CON2, CON3, CON4: value 3P-SH-SIDE -> 3P-SH-TOP; device JST:3P-SH-SIDE -> JST:3P-SH-TOP
- U5: value EFM32PG1B200F256GM32 -> EFM32GG11B520F2048GQ64; device EFM32:EFM32PG1B200F256GM32 -> EFM32:EFM32GG11B520F2048GQ64
- X1: value 40MHz -> 8MHz; device Crystal:CRYSTAL_4P -> Crystal:CRYSTAL2-SMD-5032
Connections:
- removed net SENS1: C24.C1, R19.2
- removed net SENS2: C26.C1, R21.2
- removed net SENS3: C25.C1, R20.2
- removed net SENS4: C27.C1, R22.2
- new net HSENS1: C24.C1, R19.2, U5.PD2
- new net HSENS2: C25.C1, R20.2, U5.PD3
- new net HSENS3: C26.C1, R21.2, U5.PD4
- new net HSENS4: C27.C1, R22.2, U5.PD5
- new net N$21: U5.VREGVSS
- net !BAT_CHRG: now also U5.PB4
- net !BAT_STDBY: now also U5.PB5
- net !FLASH_CS: now also U5.PE14; no longer U5.PD13
- net !RFM_CS: now also U5.PE13; no longer U5.PD12
- net 2V8: now also U5.AVDD, U5.IOVDD0@1, U5.IOVDD0@2; no longer U5.AVDD@0, U5.AVDD@1
- net 2V8_PGOOD: now also U5.PB8; no longer U5.PF3
- net GND: now also U5.VSS@1, U5.VSS@2; no longer U5.VREGVSS, X1.GND@0, X1.GND@1
- net I2C0_SCL: now also U5.PA1; no longer U5.PB15
- net I2C0_SDA: now also U5.PA0; no longer U5.PB14
- net LED: now also U5.PF5; no longer U5.PB11
- net N$16: now also U5.PB14; no longer U5.HFXTAL_N
- net N$17: now also U5.PB13; no longer U5.HFXTAL_P
- net RFM_IRQ: now also U5.PC4; no longer U5.PD14
- net RFM_RST: now also U5.PE15; no longer U5.PD15
- net US0_CLK: now also U5.PE12; no longer U5.PD9
- net US0_MISO: now also U5.PE11; no longer U5.PD11
- net US0_MOSI: now also U5.PE10; no longer U5.PD10
- net VBAT_SENSE: now also U5.PD6; no longer U5.PC11
- net VEXT_EN: now also U5.PB6
- net VEXT_PGOOD: now also U5.PB7

Commit message: Work
Parts:
- removed BAT1: 18650_CELL, Battery:18650_CELL
- added C28: 100nF, Capacitor:CAPACITOR-0603
- added CON5, CON6, CON7, CON8: 4P-SH-TOP, JST:4P-SH-TOP
- added CON9: 2P-PH-TOP, JST:2P-PH-TOP
- added R25, R26: 10K Ohms, Resistor:RESISTOR-0603
- added U9: LTC4316, Analog Devices:LTC4316
Connections:
- new net I2C0_SCL_EXT: CON5-2.S, CON6-2.S, CON7-2.S, CON8-2.S, R26.1, U9.SCLOUT
- new net I2C0_SDA_EXT: CON5-3.S, CON6-3.S, CON7-3.S, CON8-3.S, R25.1, U9.SDAOUT
- net 2V8: now also C28.C1, U9.VCC
- net GBAT: now also CON9-2.S; no longer BAT1.-
- net GND: now also C28.C2, CON5-4.S, CON6-4.S, CON7-4.S, CON8-4.S, U9.GND, U9.XORH, U9.XORL
- net I2C0_SCL: now also U9.SCLIN
- net I2C0_SDA: now also U9.SDAIN
- net VBAT: now also CON9-1.S; no longer BAT1.+
- net VEXT: now also CON5-1.S, CON6-1.S, CON7-1.S, CON8-1.S, R25.2, R26.2
- net VEXT_EN: now also U9.ENABLE

Commit message: pcb work
Parts:
- removed D1: SMAJ5.0A, TVS:SMAJ5.0A
- removed D2: B0530W, Generic Diode:B0530W
- removed F1: 1A Hold, PTC Fuses:PTC1206
- removed Q1: AO3401, Alpha Omega:AO3401
- removed R1, R3: 5.1K Ohms, Resistor:RESISTOR-0603
- removed R60, R61, R9: 100K Ohms, Resistor:RESISTOR-0603
- removed R62: 1.5K Ohms, Resistor:RESISTOR-0603
- removed U15: TP4056, TP4056:TP4056
- removed USB1: USB-C-16P-SMD-FLAT-SIDE, USB Connector:USB-C-16P-SMD-FLAT-SIDE
- C2: value 100uF -> 100nF; device Capacitor:CAPACITOR-1206 -> Capacitor:CAPACITOR-0603
- C4, C5: value 10uF -> 100nF
- U5: value EFM32GG11B520F2048GQ64 -> EFM32PG1B200F256GM32; device EFM32:EFM32GG11B520F2048GQ64 -> EFM32:EFM32PG1B200F256GM32
- X1: value 8MHz -> 40MHz; device Crystal:CRYSTAL2-SMD-5032 -> Crystal:CRYSTAL_4P
Connections:
- removed net !BAT_CHRG: R60.1, U15.!CHRG, U5.PB4
- removed net !BAT_STDBY: R61.1, U15.!STDBY, U5.PB5
- removed net 2V8_PGOOD: R9.1, U2.PG, U5.PB8
- removed net 5V0: C2.C1, D1.C, D2.A, F1.1, Q1.G, U15.CE, U15.VCC
- removed net N$21: U5.VREGVSS
- removed net N$3: R1.2, USB1.CC2
- removed net N$4: F1.2, USB1.VBUS
- removed net N$46: R62.2, U15.PROG
- removed net N$5: R3.2, USB1.CC1
- removed net VIN: C4.C1, C5.C1, C7.C1, D2.C, Q1.S, U2.EN, U2.VIN@0, U2.VIN@1
- net !FLASH_CS: now also U5.PD13; no longer U5.PE14
- net !RFM_CS: now also U5.PD12; no longer U5.PE13
- net 2V8: now also U5.AVDD@0, U5.AVDD@1; no longer R60.2, R61.2, R9.2, U5.AVDD, U5.IOVDD0@1, U5.IOVDD0@2
- net GND: now also U5.VREGVSS, X1.GND@0, X1.GND@1; no longer D1.A, R1.1, R3.1, R62.1, U15.GND@0, U15.GND@1, U15.TEMP, U5.VSS@1, U5.VSS@2, USB1.GND, USB1.SHIELD@0, USB1.SHIELD@1, USB1.SHIELD@2, USB1.SHIELD@3
- net HSENS1: now also U5.PB11; no longer U5.PD2
- net HSENS2: now also U5.PB12; no longer U5.PD3
- net HSENS3: now also U5.PB13; no longer U5.PD4
- net HSENS4: now also U5.PB14; no longer U5.PD5
- net I2C0_SCL: now also U5.PD9; no longer U5.PA1
- net I2C0_SDA: now also U5.PD10; no longer U5.PA0
- net LED: now also U5.PF3; no longer U5.PF5
- net N$16: now also U5.HFXTAL_N; no longer U5.PB14
- net N$17: now also U5.HFXTAL_P; no longer U5.PB13
- net RFM_IRQ: now also U5.PD14; no longer U5.PC4
- net RFM_RST: now also U5.PD15; no longer U5.PE15
- net US0_CLK: now also U5.PA1; no longer U5.PE12
- net US0_MISO: now also U5.PD11; no longer U5.PE11
- net US0_MOSI: now also U5.PA0; no longer U5.PE10
- net VBAT: now also U2.EN, U2.VIN@0, U2.VIN@1; no longer Q1.D, U15.BAT
- net VBAT_SENSE: now also U5.PB15; no longer U5.PD6
- net VEXT: now also C2.C1, C4.C1, C5.C1, C7.C1
- net VEXT_EN: now also U5.PC11; no longer U5.PB6
- net VEXT_PGOOD: now also U5.PC10; no longer U5.PB7
Other:
- moved on the sheet: C1, C10, C19, C21, C22, C23, C3, C6, C8, C9, CON9-1, CON9-2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

Commit message: PCB Work
Parts:
- removed R24: 330 Ohms, Resistor:RESISTOR-0603
- removed R25, R26: 10K Ohms, Resistor:RESISTOR-0603
- added R1, R3: 100K Ohms, Resistor:RESISTOR-0603
- added R9: 10M Ohm, Resistor:RESISTOR-0603
- C1: value 100nF -> 10uF
- C19: value 10uF -> 100nF
- C22: value 1uF -> 470pF
- C23: value 10uF -> 470pF
- C24, C25: value 470pF -> 100nF
- C3: value 100uF -> 100nF; device Capacitor:CAPACITOR-1206 -> Capacitor:CAPACITOR-0603
- C4: value 100nF -> 100uF; device Capacitor:CAPACITOR-0603 -> Capacitor:CAPACITOR-1206
- C5: value 100nF -> 1uF
- C6: value 470pF -> 10uF
- C7: value 100nF -> 470pF
- CON1: value 3P-SH-TOP -> 2P-PH-TOP; device JST:3P-SH-TOP -> JST:2P-PH-TOP
- CON5: value 4P-SH-TOP -> 3P-SH-TOP; device JST:4P-SH-TOP -> JST:3P-SH-TOP
- CON9: value 2P-PH-TOP -> 4P-SH-TOP; device JST:2P-PH-TOP -> JST:4P-SH-TOP
- R10: value 324K Ohms -> 100K Ohms
- R11: value 91K Ohms -> 100K Ohms
- R12: value 10M Ohm -> 10K Ohms
- R13, R23: value 100K Ohms -> 10K Ohms
- R14: value 10K Ohms -> 330 Ohms
- R15: value 10K Ohms -> 100K Ohms
- R18: value 100K Ohms -> 0 Ohms
- R22: value 0 Ohms -> 10K Ohms
- R5: value 100K Ohms -> 1K Ohms
- R6: value 100K Ohms -> 100 Ohms
- R7: value 1K Ohms -> 324K Ohms
- R8: value 100 Ohms -> 91K Ohms
- renumbered D3 to D1
Connections:
- net !FLASH_CS: now also R15.1; no longer R16.1
- net !RFM_CS: now also R17.1; no longer R18.1
- net !RST: now also R10.1; no longer R13.1
- net 2V8: now also C21.C1, R12.2, R17.2, R7.2; no longer C20.C1, R16.2, R18.2, R24.2
- net GBAT: now also CON1-2.S, R9.2; no longer CON9-2.S, R12.2
- net GND: now also C22.C2, CON5-3.S, CON9-4.S, R1.1, R16.1, R5.1, R8.1, R9.1; no longer C5.C2, CON1-3.S, CON5-4.S, R11.1, R12.1, R17.1, R6.1, R7.1
- net HSENS1: now also C22.C1, R18.2; no longer C24.C1, R19.2
- net HSENS2: now also C23.C1, R19.2; no longer C25.C1, R20.2
- net HSENS3: now also R20.2; no longer R21.2
- net HSENS4: now also R21.2; no longer R22.2
- net I2C0_SCL: now also R13.1; no longer R15.1
- net I2C0_SCL_EXT: now also CON9-2.S, R23.1; no longer CON5-2.S, R26.1
- net I2C0_SDA: now also R12.1; no longer R14.1
- net I2C0_SDA_EXT: now also CON9-3.S, R22.1; no longer CON5-3.S, R25.1
- net LED: now also R11.2; no longer R23.2
- net N$10: now also CON5-2.S, R21.1; no longer CON4-2.S, R22.1
- net N$11: now also R11.1; no longer R23.1
- net N$13: now also R7.1, R8.2; no longer R10.1, R11.2
- net N$18: now also R14.1; no longer R24.1
- net N$2: now also C5.C2; no longer C22.C2
- net N$49: now also R6.1; no longer R8.1
- net N$50: now also R5.2; no longer R7.2
- net N$6: now also C5.C1; no longer C22.C1
- net N$7: now also CON3-2.S, R19.1; no longer CON2-2.S, R20.1
- net N$8: now also CON4-2.S, R20.1; no longer CON3-2.S, R21.1
- net N$9: now also CON2-2.S, R18.1; no longer CON1-2.S, R19.1
- net RFM_RST: now also R16.2; no longer R17.2
- net VBAT: now also C2.C1, C4.C1, CON1-1.S, R3.2, R6.2; no longer C19.C1, C21.C1, CON9-1.S, R5.2, R8.2
- net VBAT_SENSE: now also C7.C1, R3.1, R4.2; no longer C6.C1, R5.1, R6.2
- net VEXT: now also C19.C1, C20.C1, C24.C1, C25.C1, C6.C1, CON9-1.S, R22.2, R23.2; no longer C2.C1, C23.C1, C4.C1, C5.C1, C7.C1, CON1-1.S, R25.2, R26.2
- net VEXT_EN: now also R1.2; no longer R4.2
Other:
- moved on the sheet: C1, C20, C24, C25, C3, C6, CON2-1, CON2-2, CON2-3, CON3-1, CON3-2, CON3-3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

Commit message: Change DRCs
Parts:
- added LOGO1: JS-5MM, Silkscreen:JS-5MM
Changed lines of the file:
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@@
 <part name="C20" library="Capacitor" deviceset="CAPACITOR" device="-0603" value="100nF"/>
 <part name="GND36" library="Supply Symbol" deviceset="GND" device=""/>
+<part name="LOGO1" library="Silkscreen" deviceset="JS" device="-5MM" value="JS-5MM"/>
 </parts>
 <sheets>
@@
 <attribute name="VALUE" x="14.986" y="88.9" size="1.778" layer="96"/>
 </instance>
+<instance part="LOGO1" gate="G$1" x="368.3" y="27.94" smashed="yes"/>
 </instances>
 <busses>
@@
 </drawing>
 <compatibility>
+<note version="6.3" minversion="6.2.2" severity="warning">
+Since Version 6.2.2 text objects can contain more than one line,
+which will not be processed correctly with this version.
+</note>
 <note version="8.3" severity="warning">
 Since Version 8.3, EAGLE supports URNs for individual library

Commit message: Finish board (needs revision)
Connections:
- net !FLASH_CS: now also U5.PD12; no longer U5.PD13
- net !RFM_CS: now also U5.PD13; no longer U5.PD12
Changed lines of the file:
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@@
 <part name="2V87" library="Supply Symbol" deviceset="2V8" device=""/>
 <part name="GND20" library="Supply Symbol" deviceset="GND" device=""/>
-<part name="U7" library="HopeRF" deviceset="RFM69H" device="W" value="RFM69HW"/>
+<part name="U7" library="HopeRF" deviceset="RFM69*" device="W" technology="H" value="RFM69HW"/>
 <part name="GND33" library="Supply Symbol" deviceset="GND" device=""/>
 <part name="C18" library="Capacitor" deviceset="CAPACITOR" device="-0603" value="100nF"/>
@@
 </segment>
 <segment>
-<label x="175.26" y="137.16" size="1.778" layer="95" xref="yes"/>
-<wire x1="170.18" y1="137.16" x2="175.26" y2="137.16" width="0.1524" layer="91"/>
-<pinref part="U5" gate="G$1" pin="PD13"/>
+<label x="200.66" y="139.7" size="1.778" layer="95" xref="yes"/>
+<wire x1="170.18" y1="139.7" x2="200.66" y2="139.7" width="0.1524" layer="91"/>
+<pinref part="U5" gate="G$1" pin="PD12"/>
 </segment>
 </net>
@@
 <net name="!RFM_CS" class="0">
 <segment>
-<label x="200.66" y="139.7" size="1.778" layer="95" xref="yes"/>
-<wire x1="170.18" y1="139.7" x2="200.66" y2="139.7" width="0.1524" layer="91"/>
-<pinref part="U5" gate="G$1" pin="PD12"/>
-</segment>
-</net>
+<label x="175.26" y="137.16" size="1.778" layer="95" xref="yes"/>
+<wire x1="170.18" y1="137.16" x2="175.26" y2="137.16" width="0.1524" layer="91"/>
+<pinref part="U5" gate="G$1" pin="PD13"/>
+</segment>
+</net>
