File: pcb/plant-sense.brd (EAGLE design)
At the start: 48.5 x 48.5 mm, 78 parts, among them CON1 2P-PH-TOP, CON2 3P-SH-TOP, CON3 3P-SH-TOP, CON4 3P-SH-TOP, CON5 3P-SH-TOP, CON6 4P-SH-TOP, CON7 4P-SH-TOP, CON8 4P-SH-TOP, CON9 4P-SH-TOP, T1 BC817, U1 MCP1253-33X50, U2 MIC23155, U3 FS312F-G, U4 FS8205, U5 EFM32PG1B200F256GM32, U6 SST26VF016B, U7 RFM69HW, U8 SI7021, U9 LTC4316, X1 40MHz

Commit message: Sync library updates Add schematic PDF
Connections:
- net N$15: now also D1.C; no longer D1.1
- net N$18: now also D1.A; no longer D1.2
